Commit message: fix: sửa mesh names, Caster axis, sensor links và IMU plugin cho Gazebo ROS1
Agent-Logs-Url: https://github.com/hoaiphu1002/ROS1_MELODIC_ROBOT/sessions/e1e77246-c6f3-488c-abab-3ff58971ce43

Co-authored-by: hoaiphu10022004 <198301165+hoaiphu10022004@users.noreply.github.com>

File: src/robot_fablab/urdf/robot_fablab.urdf (robot description, URDF)
Before this commit: robot reception, 8 links, 7 joints
Links:
- link link_camera: geometry collision box size=0.03 0.09 0.025; visual box size=0.03 0.09 0.025
- link link_lidar: geometry collision cylinder length=0.04 radius=0.035; visual cylinder length=0.04 radius=0.035

File: src/robot_fablab/urdf/robot_fablab.xacro (robot description, xacro)
@@ -133,5 +133,5 @@
       <origin xyz="0 0 0" rpy="0 0 0" />
       <geometry>
-        <mesh filename="package://robot_fablab/meshes/link_lidar.STL" />
+        <cylinder radius="0.035" length="0.04"/>
       </geometry>
       <material name="">
@@ -142,5 +142,5 @@
       <origin xyz="0 0 0" rpy="0 0 0" />
       <geometry>
-        <mesh filename="package://robot_fablab/meshes/link_lidar.STL" />
+        <cylinder radius="0.035" length="0.04"/>
       </geometry>
     </collision>
@@ -161,5 +161,5 @@
       <origin xyz="0 0 0" rpy="0 0 0" />
       <geometry>
-        <mesh filename="package://robot_fablab/meshes/link_camera.STL" />
+        <box size="0.03 0.09 0.025"/>
       </geometry>
       <material name="">
@@ -170,5 +170,5 @@
       <origin xyz="0 0 0" rpy="0 0 0" />
       <geometry>
-        <mesh filename="package://robot_fablab/meshes/link_camera.STL" />
+        <box size="0.03 0.09 0.025"/>
       </geometry>
     </collision>

File: src/robot_fablab/urdf/ros_f.urdf (robot description, URDF)
Before this commit: robot ros_f, 5 links, 4 joints
Links:
- added link imu_link, mass 0.01; collision box size=0.01 0.01 0.01; visual box size=0.01 0.01 0.01
- added link link_camera, mass 0.15; collision box size=0.03 0.09 0.025; visual box size=0.03 0.09 0.025
- added link link_lidar, mass 0.035; collision cylinder length=0.04 radius=0.035; visual cylinder length=0.04 radius=0.035
- link Caster: geometry collision mesh filename=package://robot_fablab/meshes/Caster.STL; visual mesh filename=package://robot_fablab/meshes/Caster.STL
- link Left_wheel: geometry collision mesh filename=package://robot_fablab/meshes/Left_wheel.STL; visual mesh filename=package://robot_fablab/meshes/Left_wheel.STL
- link Right_wheel: geometry collision mesh filename=package://robot_fablab/meshes/Right_wheel.STL; visual mesh filename=package://robot_fablab/meshes/Right_wheel.STL
Joints:
- added joint imu_joint: type fixed, parent base_link, child imu_link, origin xyz=0 0 0 rpy=0 0 0
- added joint joint_camera: type fixed, parent base_link, child link_camera, origin xyz=-0.11803 0.012232 1.3955 rpy=0 0 0, axis 0 0 0
- added joint joint_lidar: type fixed, parent base_link, child link_lidar, origin xyz=0.011534 0.010999 0.55646 rpy=0 0 0, axis 0 0 0
- joint Caster_joint: axis 0 0 0 -> 0 0 1
