Commit message: Configure gazebo simulation to use ros_f.urdf robot model
Agent-Logs-Url: https://github.com/hoaiphu1002/ROS1_MELODIC_ROBOT/sessions/91fc9ba4-7d84-4446-b8cd-a335e5e70c3d

Co-authored-by: hoaiphu10022004 <198301165+hoaiphu10022004@users.noreply.github.com>

File: src/robot_fablab/urdf/ros_f.urdf (robot description, URDF)
Before this commit: robot ros_f, 4 links, 3 joints
Links:
- added link base_footprint; visual box size=0.001 0.001 0.001
- link Caster: geometry collision mesh filename=package://robot_fablab/meshes/link_caster.STL; visual mesh filename=package://robot_fablab/meshes/link_caster.STL
- link Left_wheel: geometry collision mesh filename=package://robot_fablab/meshes/link_left.STL; visual mesh filename=package://robot_fablab/meshes/link_left.STL
- link Right_wheel: geometry collision mesh filename=package://robot_fablab/meshes/link_right.STL; visual mesh filename=package://robot_fablab/meshes/link_right.STL
- link base_link: geometry collision mesh filename=package://robot_fablab/meshes/base_link.STL; visual mesh filename=package://robot_fablab/meshes/base_link.STL
Joints:
- added joint base_footprint_joint: type fixed, parent base_footprint, child base_link, origin xyz=0 0 0 rpy=0 0 0

Commit message: Use ros_f.urdf in gazebo simulation with cmd_vel support
Agent-Logs-Url: https://github.com/hoaiphu1002/ROS1_MELODIC_ROBOT/sessions/29f6b418-3930-42ca-8dc8-7d279e88b9d3

Co-authored-by: hoaiphu10022004 <198301165+hoaiphu10022004@users.noreply.github.com>

File: src/robot_fablab/urdf/ros_f.urdf (robot description, URDF)
Before this commit: robot ros_f, 4 links, 3 joints
Links:
- link Caster: geometry collision mesh filename=package://robot_fablab/meshes/link_caster.STL; visual mesh filename=package://robot_fablab/meshes/link_caster.STL
- link Left_wheel: geometry collision mesh filename=package://robot_fablab/meshes/link_left.STL; visual mesh filename=package://robot_fablab/meshes/link_left.STL
- link Right_wheel: geometry collision mesh filename=package://robot_fablab/meshes/link_right.STL; visual mesh filename=package://robot_fablab/meshes/link_right.STL
- link base_link: geometry collision mesh filename=package://robot_fablab/meshes/base_link.STL; visual mesh filename=package://robot_fablab/meshes/base_link.STL

Commit message: Update gazebo.launch to use ros_f.urdf and fix URDF for Gazebo compatibility
Agent-Logs-Url: https://github.com/hoaiphu1002/ROS1_MELODIC_ROBOT/sessions/fb3cf776-3f62-45a3-8f1a-8046e5d8ebd9

Co-authored-by: hoaiphu10022004 <198301165+hoaiphu10022004@users.noreply.github.com>

File: src/robot_fablab/urdf/ros_f.urdf (robot description, URDF)
Before this commit: robot ros_f, 4 links, 3 joints
Links:
- added link base_footprint
- link Caster: geometry collision mesh filename=package://robot_fablab/meshes/link_caster.STL; visual mesh filename=package://robot_fablab/meshes/link_caster.STL
- link Left_wheel: geometry collision mesh filename=package://robot_fablab/meshes/link_left.STL; visual mesh filename=package://robot_fablab/meshes/link_left.STL
- link Right_wheel: geometry collision mesh filename=package://robot_fablab/meshes/link_right.STL; visual mesh filename=package://robot_fablab/meshes/link_right.STL
- link base_link: geometry collision mesh filename=package://robot_fablab/meshes/base_link.STL; visual mesh filename=package://robot_fablab/meshes/base_link.STL
Joints:
- removed joint Left_wheel_joint
- removed joint Right_wheel_joint
- added joint base_footprint_joint: type fixed, parent base_footprint, child base_link, origin xyz=0 0 0 rpy=0 0 0
- added joint joint_left: type continuous, parent base_link, child Left_wheel, origin xyz=0.71544 0.76308 -0.015158 rpy=0 0 -3.1416, axis 0 1 0
- added joint joint_right: type continuous, parent base_link, child Right_wheel, origin xyz=0.71544 0.18036 -0.015158 rpy=0 0 3.1416, axis 0 -1 0
- joint Caster_joint: axis 0 0 0 -> 0 0 1

Commit message: fix: align all config/launch files with ros_f.urdf as single source of truth
Agent-Logs-Url: https://github.com/hoaiphu1002/ROS1_MELODIC_ROBOT/sessions/ce2d0624-9431-4890-8c66-ced96d406119

Co-authored-by: hoaiphu10022004 <198301165+hoaiphu10022004@users.noreply.github.com>

File: src/robot_fablab/urdf/ros_f.urdf (robot description, URDF)
Before this commit: robot ros_f, 5 links, 4 joints
Links:
- added link imu_link, mass 0.01; collision box size=0.01 0.01 0.01; visual box size=0.01 0.01 0.01
- added link link_camera, mass 0.15; collision box size=0.05 0.12 0.035; visual box size=0.05 0.12 0.035
- added link link_lidar, mass 0.035; collision cylinder length=0.04 radius=0.05; visual cylinder length=0.04 radius=0.05
- link Caster: geometry collision mesh filename=package://robot_fablab/meshes/Caster.STL; visual mesh filename=package://robot_fablab/meshes/Caster.STL
- link Left_wheel: geometry collision mesh filename=package://robot_fablab/meshes/Left_wheel.STL; visual mesh filename=package://robot_fablab/meshes/Left_wheel.STL
- link Right_wheel: geometry collision mesh filename=package://robot_fablab/meshes/Right_wheel.STL; visual mesh filename=package://robot_fablab/meshes/Right_wheel.STL
Joints:
- added joint imu_joint: type fixed, parent base_link, child imu_link, origin xyz=0.5 0.47172 0.1 rpy=0 0 0
- added joint joint_camera: type fixed, parent base_link, child link_camera, origin xyz=0.0 0.47172 0.7 rpy=0 0 0, axis 0 0 0
- added joint joint_lidar: type fixed, parent base_link, child link_lidar, origin xyz=0.3 0.47172 0.4 rpy=0 0 0, axis 0 0 0
