Commit message: fix: fix all Gazebo simulation issues for ROS1 Melodic
Agent-Logs-Url: https://github.com/hoaiphu1002/ROS1_MELODIC_ROBOT/sessions/bb6cbb8c-e85b-42ea-9b86-743ec75d98d4

Co-authored-by: hoaiphu10022004 <198301165+hoaiphu10022004@users.noreply.github.com>

File: src/robot_fablab/urdf/robot_fablab.xacro (robot description, xacro)
@@ -133,5 +133,5 @@
       <origin xyz="0 0 0" rpy="0 0 0" />
       <geometry>
-        <mesh filename="package://robot_fablab/meshes/link_lidar.STL" />
+        <cylinder radius="0.05" length="0.04"/>
       </geometry>
       <material name="">
@@ -142,5 +142,5 @@
       <origin xyz="0 0 0" rpy="0 0 0" />
       <geometry>
-        <mesh filename="package://robot_fablab/meshes/link_lidar.STL" />
+        <cylinder radius="0.05" length="0.04"/>
       </geometry>
     </collision>
@@ -161,5 +161,5 @@
       <origin xyz="0 0 0" rpy="0 0 0" />
       <geometry>
-        <mesh filename="package://robot_fablab/meshes/link_camera.STL" />
+        <box size="0.05 0.12 0.035"/>
       </geometry>
       <material name="">
@@ -170,5 +170,5 @@
       <origin xyz="0 0 0" rpy="0 0 0" />
       <geometry>
-        <mesh filename="package://robot_fablab/meshes/link_camera.STL" />
+        <box size="0.05 0.12 0.035"/>
       </geometry>
     </collision>

Commit message: ok

File: src/robot_fablab/urdf/robot_fablab.xacro (robot description, xacro)
@@ -1,6 +1,7 @@
-<?xml version='1.0'?>
-<robot name="reception"
-  xmlns:xacro="http://www.ros.org/wiki/xacro">
+<?xml version="1.0" encoding="utf-8"?>
+<robot name="reception" xmlns:xacro="http://www.ros.org/wiki/xacro">
+  <!-- 1. Include Gazebo plugins -->
   <xacro:include filename="$(find robot_fablab)/urdf/robot_fablab.gazebo"/>
+  <!-- ================= BASE FOOTPRINT ================= -->
   <link name="base_footprint">
     <visual>
@@ -15,36 +16,38 @@
     <origin xyz="0 0 0" rpy="0 0 0"/>
   </joint>
+  <!-- ================= BASE LINK ================= -->
   <link name="base_link">
     <inertial>
-      <origin xyz="-0.025807 0.027971 0.41357" rpy="0 0 0" />
-      <mass value="29.924" />
-      <inertia ixx="1.0006" ixy="-0.0013232" ixz="0.0065325" iyy="0.70301" iyz="-3.0656E-05" izz="1.3855" />
-    </inertial>
-    <visual>
-      <origin xyz="0 0 0" rpy="0 0 0" />
-      <geometry>
-        <mesh filename="package://robot_fablab/meshes/base_link.STL" />
-      </geometry>
-      <material name="">
-        <color rgba="0.79216 0.81961 0.93333 1" />
-      </material>
-    </visual>
-    <collision>
-      <origin xyz="0 0 0" rpy="0 0 0" />
-      <geometry>
-        <mesh filename="package://robot_fablab/meshes/base_link.STL" />
-      </geometry>
-    </collision>
-  </link>
-  <link name="link_left">
-    <inertial>
-      <origin xyz="-0.00011936 0.00025083 0.014883" rpy="0 0 0" />
-      <mass value="1.0707" />
-      <inertia ixx="0.0032566" ixy="1.1489E-08" ixz="-1.3959E-05" iyy="0.0032564" iyz="-9.4568E-09" izz="0.0062144" />
-    </inertial>
-    <visual>
-      <origin xyz="0 0 0" rpy="0 0 0" />
-      <geometry>
-        <cylinder radius="0.1" length="0.05"/>
+      <origin xyz="0.80547 0.29964 -0.47356" rpy="0 0 0" />
+      <mass value="13.533" />
+      <inertia ixx="0.22773" ixy="-0.0049825" ixz="5.9491E-05" iyy="0.3509" iyz="5.9312E-05" izz="0.14899" />
+    </inertial>
+    <visual>
+      <origin xyz="0 0 0" rpy="0 0 0" />
+      <geometry>
+        <mesh filename="package://robot_fablab/meshes1/base_link.STL" />
+      </geometry>
+      <material name="">
+        <color rgba="0.74902 0.74902 0.74902 1" />
+      </material>
+    </visual>
+    <collision>
+      <origin xyz="0 0 0" rpy="0 0 0" />
+      <geometry>
+        <mesh filename="package://robot_fablab/meshes1/base_link.STL" />
+      </geometry>
+    </collision>
+  </link>
+  <!-- ================= WHEELS ================= -->
+  <link name="Left_wheel">
+    <inertial>
+      <origin xyz="-0.00025563 0.014871 7.2657E-07" rpy="0 0 0" />
+      <mass value="1.0716" />
+      <inertia ixx="0.0032564" ixy="1.521E-09" ixz="-6.2778E-09" iyy="0.0062145" iyz="4.2157E-08" izz="0.0032565" />
+    </inertial>
+    <visual>
+      <origin xyz="0 0 0" rpy="0 0 0" />
+      <geometry>
+        <mesh filename="package://robot_fablab/meshes1/Left_wheel.STL" />
       </geometry>
       <material name="">
@@ -55,25 +58,25 @@
       <origin xyz="0 0 0" rpy="0 0 0" />
       <geometry>
-        <cylinder radius="0.1" length="0.05"/>
-      </geometry>
-    </collision>
-  </link>
-  <joint name="joint_left" type="continuous">
-    <origin xyz="0.19672 0.3411 0.036748" rpy="1.5708 0 0" />
-    <parent link="base_link" />
-    <child link="link_left" />
-    <axis xyz="0 0 -1" />
+        <mesh filename="package://robot_fablab/meshes1/Left_wheel.STL" />
+      </geometry>
+    </collision>
+  </link>
+  <joint name="Left_wheel_joint" type="continuous">
+    <origin xyz="0.71544 0.76308 -0.015158" rpy="0 0 -3.1416" />
+    <parent link="base_link" />
+    <child link="Left_wheel" />
+    <axis xyz="0 1 0" />
     <dynamics damping="0.1" friction="0.1" />
   </joint>
-  <link name="link_right">
-    <inertial>
-      <origin xyz="0.00023152 0.00019816 -0.014882" rpy="0 0 0" />
-      <mass value="1.0707" />
-      <inertia ixx="0.0032565" ixy="-4.4065E-08" ixz="-1.3949E-05" iyy="0.0032564" iyz="2.7514E-08" izz="0.0062144" />
-    </inertial>
-    <visual>
-      <origin xyz="0 0 0" rpy="0 0 0" />
-      <geometry>
-        <cylinder radius="0.1" length="0.05"/>
+  <link name="Right_wheel">
+    <inertial>
+      <origin xyz="-0.00025564 -0.014871 7.261E-07" rpy="0 0 0" />
+      <mass value="1.0716" />
+      <inertia ixx="0.0032564" ixy="-1.5005E-09" ixz="-6.3105E-09" iyy="0.0062145" iyz="-4.2151E-08" izz="0.0032565" />
+    </inertial>
+    <visual>
+      <origin xyz="0 0 0" rpy="0 0 0" />
+      <geometry>
+        <mesh filename="package://robot_fablab/meshes1/Right_wheel.STL" />
       </geometry>
       <material name="">
@@ -84,44 +87,46 @@
       <origin xyz="0 0 0" rpy="0 0 0" />
       <geometry>
-        <cylinder radius="0.1" length="0.05"/>
-      </geometry>
-    </collision>
-  </link>
-  <joint name="joint_right" type="continuous">
-    <origin xyz="0.1933 -0.34091 0.0368" rpy="1.5708 0 0" />
-    <parent link="base_link" />
-    <child link="link_right" />
-    <axis xyz="0 0 -1" />
+        <mesh filename="package://robot_fablab/meshes1/Right_wheel.STL" />
+      </geometry>
+    </collision>
+  </link>
+  <joint name="Right_wheel_joint" type="continuous">
+    <origin xyz="0.71544 0.18036 -0.015158" rpy="0 0 3.1416" />
+    <parent link="base_link" />
+    <child link="Right_wheel" />
+    <axis xyz="0 -1 0" />
     <dynamics damping="0.1" friction="0.1" />
   </joint>
-  <link name="link_caster">
-    <inertial>
-      <origin xyz="0.018731 0.021844 -0.00013927" rpy="0 0 0" />
-      <mass value="0.37837" />
-      <inertia ixx="0.00048693" ixy="-8.3984E-05" ixz="2.0261E-06" iyy="0.00045028" iyz="1.5693E-06" izz="0.00064534" />
-    </inertial>
-    <visual>
-      <origin xyz="0 0 0" rpy="0 0 0" />
-      <geometry>
-        <sphere radius="0.038"/>
-      </geometry>
-      <material name="">
-        <color rgba="0.79216 0.81961 0.93333 1" />
-      </material>
-    </visual>
-    <collision>
-      <origin xyz="0 0 0" rpy="0 0 0" />
-      <geometry>
-        <sphere radius="0.04"/>
-      </geometry>
-    </collision>
-  </link>
-  <joint name="joint_caster" type="continuous">
-    <origin xyz="-0.25394 0.00080362 -0.0255" rpy="1.5708 0 0" />
-    <parent link="base_link" />
-    <child link="link_caster" />
-    <axis xyz="0 0 1" />
-    <dynamics damping="0.1" friction="0.1" />
-  </joint>
+  <link name="Caster">
+    <inertial>
+      <origin xyz="-0.00326890758980913 -0.000105769701198966 -0.0476560909473075" rpy="0 0 0" />
+      <mass value="0.378365009719551" />
+      <inertia ixx="0.000486902921012301" ixy="4.68634433031941E-08" ixz="-8.39976891943837E-05" iyy="0.000645365810716879" iyz="-4.71799768324587E-07" izz="0.000450276858110533" />
+    </inertial>
+    <visual>
+      <origin xyz="0 0 0" rpy="0 0 0" />
+      <geometry>
+        <mesh filename="package://robot_fablab/meshes1/Caster.STL" />
+      </geometry>
+      <material name="">
+        <color rgba="0.792156862745098 0.819607843137255 0.933333333333333 1" />
+      </material>
+    </visual>
+    <collision>
+      <origin xyz="0 0 0" rpy="0 0 0" />
+      <geometry>
+        <mesh filename="package://robot_fablab/meshes1/Caster.STL" />
+      </geometry>
+    </collision>
+  </link>
+  <joint name="Caster_joint" type="continuous">
+    <origin xyz="1.0482 0.47172 -0.0081577" rpy="0 0 -3.1416" />
+    <parent link="base_link" />
+    <child link="Caster" />
+    <axis xyz="0 1 0" />  <!-- fixed axis from 0 0 0 to 0 1 0 -->
+    <dynamics damping="0.01" friction="0.01" />
+  </joint>
+  <!-- ================= SENSORS ================= -->
+  <!-- Lidar -->
   <link name="link_lidar">
     <inertial>
@@ -133,5 +138,5 @@
       <origin xyz="0 0 0" rpy="0 0 0" />
       <geometry>
-        <mesh filename="package://robot_fablab/meshes/link_lidar.STL" />
+        <mesh filename="package://robot_fablab/meshes1/link_lidar.STL" />
       </geometry>
       <material name="">
@@ -142,5 +147,5 @@
       <origin xyz="0 0 0" rpy="0 0 0" />
       <geometry>
-        <mesh filename="package://robot_fablab/meshes/link_lidar.STL" />
+        <mesh filename="package://robot_fablab/meshes1/link_lidar.STL" />
       </geometry>
     </collision>
@@ -152,4 +157,5 @@
     <axis xyz="0 0 0" />
   </joint>
+  <!-- Camera -->
   <link name="link_camera">
     <inertial>
@@ -161,5 +167,5 @@
       <origin xyz="0 0 0" rpy="0 0 0" />
       <geometry>
-        <mesh filename="package://robot_fablab/meshes/link_camera.STL" />
+        <mesh filename="package://robot_fablab/meshes1/link_camera.STL" />
       </geometry>
       <material name="">
@@ -170,5 +176,5 @@
       <origin xyz="0 0 0" rpy="0 0 0" />
       <geometry>
-        <mesh filename="package://robot_fablab/meshes/link_camera.STL" />
+        <mesh filename="package://robot_fablab/meshes1/link_camera.STL" />
       </geometry>
     </collision>
@@ -180,4 +186,5 @@
     <axis xyz="0 0 0" />
   </joint>
+  <!-- IMU -->
   <link name="imu_link">
     <visual>
@@ -207,24 +214,24 @@
     <origin xyz="0 0 0" rpy="0 0 0"/>
   </joint>
-  <!-- transmission -->
+  <!-- ================= TRANSMISSION GAZEBO CONTROL ================= -->
   <transmission name="right_wheel_trans">
     <type>transmission_interface/SimpleTransmission</type>
+    <joint name="Right_wheel_joint">
+      <hardwareInterface>hardware_interface/VelocityJointInterface</hardwareInterface>
+    </joint>
     <actuator name="motor_right_wheel">
-      <hardwareInterface>EffortJointInterface</hardwareInterface>
+      <hardwareInterface>hardware_interface/VelocityJointInterface</hardwareInterface>
       <mechanicalReduction>1</mechanicalReduction>
     </actuator>
-    <joint name="joint_right">
-      <hardwareInterface>VelocityJointInterface</hardwareInterface>
-    </joint>
   </transmission>
   <transmission name="left_wheel_trans">
     <type>transmission_interface/SimpleTransmission</type>
+    <joint name="Left_wheel_joint">
+      <hardwareInterface>hardware_interface/VelocityJointInterface</hardwareInterface>
+    </joint>
     <actuator name="motor_left_wheel">
-      <hardwareInterface>EffortJointInterface</hardwareInterface>
+      <hardwareInterface>hardware_interface/VelocityJointInterface</hardwareInterface>
       <mechanicalReduction>1</mechanicalReduction>
     </actuator>
-    <joint name="joint_left">
-      <hardwareInterface>VelocityJointInterface</hardwareInterface>
-    </joint>
   </transmission>
 </robot>

Commit message: okok

File: src/robot_fablab/urdf/robot_fablab.xacro (robot description, xacro)
@@ -28,6 +28,7 @@
         <mesh filename="package://robot_fablab/meshes1/base_link.STL" />
       </geometry>
-      <material name="">
-        <color rgba="0.74902 0.74902 0.74902 1" />
+      <!-- force base_link to white in URDF -->
+      <material name="white">
+        <color rgba="1 1 1 1" />
       </material>
     </visual>
@@ -124,5 +125,5 @@
     <parent link="base_link" />
     <child link="Caster" />
-    <axis xyz="0 1 0" />  <!-- fixed axis from 0 0 0 to 0 1 0 -->
+    <axis xyz="0 1 0" />
     <dynamics damping="0.01" friction="0.01" />
   </joint>
@@ -155,33 +156,4 @@
     <parent link="base_link" />
     <child link="link_lidar" />
-    <axis xyz="0 0 0" />
-  </joint>
-  <!-- Camera -->
-  <link name="link_camera">
-    <inertial>
-      <origin xyz="-0.016107 4.0071E-05 -0.00053431" rpy="0 0 0" />
-      <mass value="0.15226" />
-      <inertia ixx="0.0003084" ixy="-1.3455E-06" ixz="-4.4401E-08" iyy="2.2766E-05" iyz="9.3764E-09" izz="0.00031076" />
-    </inertial>
-    <visual>
-      <origin xyz="0 0 0" rpy="0 0 0" />
-      <geometry>
-        <mesh filename="package://robot_fablab/meshes1/link_camera.STL" />
-      </geometry>
-      <material name="">
-        <color rgba="0.27059 0.27059 0.27059 1" />
-      </material>
-    </visual>
-    <collision>
-      <origin xyz="0 0 0" rpy="0 0 0" />
-      <geometry>
-        <mesh filename="package://robot_fablab/meshes1/link_camera.STL" />
-      </geometry>
-    </collision>
-  </link>
-  <joint name="joint_camera" type="fixed">
-    <origin xyz="-0.11803 0.012232 1.3955" rpy="0 0 0" />
-    <parent link="base_link" />
-    <child link="link_camera" />
     <axis xyz="0 0 0" />
   </joint>

Commit message: ok

File: src/robot_fablab/urdf/robot_fablab.xacro (robot description, xacro)
@@ -2,5 +2,5 @@
 <robot name="reception" xmlns:xacro="http://www.ros.org/wiki/xacro">
   <!-- 1. Include Gazebo plugins -->
-  <xacro:include filename="$(find robot_fablab)/urdf/robot_fablab.gazebo"/>
+  <xacro:include filename="$(find robot_fablab)/urdf/robot_datn.gazebo"/>
   <!-- ================= BASE FOOTPRINT ================= -->
   <link name="base_footprint">
@@ -28,5 +28,4 @@
         <mesh filename="package://robot_fablab/meshes1/base_link.STL" />
       </geometry>
-      <!-- force base_link to white in URDF -->
       <material name="white">
         <color rgba="1 1 1 1" />
@@ -40,5 +39,5 @@
     </collision>
   </link>
-  <!-- ================= WHEELS ================= -->
+  <!-- ================= WHEELS (giong code cu: cylinder) ================= -->
   <link name="Left_wheel">
     <inertial>
@@ -48,7 +47,7 @@
     </inertial>
     <visual>
-      <origin xyz="0 0 0" rpy="0 0 0" />
+      <origin xyz="0 0 0" rpy="1.5708 0 0" />
       <geometry>
-        <mesh filename="package://robot_fablab/meshes1/Left_wheel.STL" />
+        <cylinder radius="0.1" length="0.05"/>
       </geometry>
       <material name="">
@@ -57,12 +56,12 @@
     </visual>
     <collision>
-      <origin xyz="0 0 0" rpy="0 0 0" />
+      <origin xyz="0 0 0" rpy="1.5708 0 0" />
       <geometry>
-        <mesh filename="package://robot_fablab/meshes1/Left_wheel.STL" />
+        <cylinder radius="0.1" length="0.05"/>
       </geometry>
     </collision>
   </link>
   <joint name="Left_wheel_joint" type="continuous">
-    <origin xyz="0.71544 0.76308 -0.015158" rpy="0 0 -3.1416" />
+    <origin xyz="0.71544 0.76308 -0.015158" rpy="0 0 0" />
     <parent link="base_link" />
     <child link="Left_wheel" />
@@ -77,7 +76,7 @@
     </inertial>
     <visual>
-      <origin xyz="0 0 0" rpy="0 0 0" />
+      <origin xyz="0 0 0" rpy="1.5708 0 0" />
       <geometry>
-        <mesh filename="package://robot_fablab/meshes1/Right_wheel.STL" />
+        <cylinder radius="0.1" length="0.05"/>
       </geometry>
       <material name="">
@@ -86,27 +85,29 @@
     </visual>
     <collision>
-      <origin xyz="0 0 0" rpy="0 0 0" />
+      <origin xyz="0 0 0" rpy="1.5708 0 0" />
       <geometry>
-        <mesh filename="package://robot_fablab/meshes1/Right_wheel.STL" />
+        <cylinder radius="0.1" length="0.05"/>
       </geometry>
     </collision>
   </link>
   <joint name="Right_wheel_joint" type="continuous">
-    <origin xyz="0.71544 0.18036 -0.015158" rpy="0 0 3.1416" />
+    <origin xyz="0.71544 0.18036 -0.015158" rpy="0 0 0" />
     <parent link="base_link" />
     <child link="Right_wheel" />
-    <axis xyz="0 -1 0" />
+    <axis xyz="0 1 0" />
     <dynamics damping="0.1" friction="0.1" />
   </joint>
+  <!-- ================= CASTER ================= -->
   <link name="Caster">
     <inertial>
       <origin xyz="-0.00326890758980913 -0.000105769701198966 -0.0476560909473075" rpy="0 0 0" />
       <mass value="0.378365009719551" />
-      <inertia ixx="0.000486902921012301" ixy="4.68634433031941E-08" ixz="-8.39976891943837E-05" iyy="0.000645365810716879" iyz="-4.71799768324587E-07" izz="0.000450276858110533" />
+      <inertia ixx="0.000486902921012301" ixy="4.68634433031941E-08" ixz="-8.39976891943837E-05"
+               iyy="0.000645365810716879" iyz="-4.71799768324587E-07" izz="0.000450276858110533" />
     </inertial>
     <visual>
-      <origin xyz="0 0 0" rpy="0 0 0" />
+      <origin xyz="0 0 -0.115158" rpy="0 0 0" />
       <geometry>
-        <mesh filename="package://robot_fablab/meshes1/Caster.STL" />
+        <sphere radius="0.038"/>
       </geometry>
       <material name="">
@@ -115,48 +116,18 @@
     </visual>
     <collision>
-      <origin xyz="0 0 0" rpy="0 0 0" />
+      <origin xyz="0 0 -0.115158" rpy="0 0 0" />
       <geometry>
-        <mesh filename="package://robot_fablab/meshes1/Caster.STL" />
+        <sphere radius="0.04"/>
       </geometry>
     </collision>
   </link>
   <joint name="Caster_joint" type="continuous">
-    <origin xyz="1.0482 0.47172 -0.0081577" rpy="0 0 -3.1416" />
+    <!-- FIX: only changed Z from -0.0081577 to 0.04 -->
+    <origin xyz="1.0482 0.47172 0.04" rpy="0 0 3.1416" />
     <parent link="base_link" />
     <child link="Caster" />
-    <axis xyz="0 1 0" />
-    <dynamics damping="0.01" friction="0.01" />
+    <axis xyz="0 0 1" />
+    <dynamics damping="0.1" friction="0.1" />
   </joint>
-  <!-- ================= SENSORS ================= -->
-  <!-- Lidar -->
-  <link name="link_lidar">
-    <inertial>
-      <origin xyz="-0.002487 1.09E-05 -0.024095" rpy="0 0 0" />
-      <mass value="0.035081" />
-      <inertia ixx="1.9431E-05" ixy="7.3718E-10" ixz="4.0724E-08" iyy="1.932E-05" iyz="-1.091E-09" izz="3.7018E-05" />
-    </inertial>
-    <visual>
-      <origin xyz="0 0 0" rpy="0 0 0" />
-      <geometry>
-        <mesh filename="package://robot_fablab/meshes1/link_lidar.STL" />
-      </geometry>
-      <material name="">
-        <color rgba="0 0 0 1" />
-      </material>
-    </visual>
-    <collision>
-      <origin xyz="0 0 0" rpy="0 0 0" />
-      <geometry>
-        <mesh filename="package://robot_fablab/meshes1/link_lidar.STL" />
-      </geometry>
-    </collision>
-  </link>
-  <joint name="joint_lidar" type="fixed">
-    <origin xyz="0.011534 0.010999 0.55646" rpy="0 0 0" />
-    <parent link="base_link" />
-    <child link="link_lidar" />
-    <axis xyz="0 0 0" />
-  </joint>
-  <!-- IMU -->
   <link name="imu_link">
     <visual>
@@ -169,10 +140,4 @@
       </material>
     </visual>
-    <collision>
-      <origin xyz="0 0 0" rpy="0 0 0"/>
-      <geometry>
-        <box size="0.01 0.01 0.01"/>
-      </geometry>
-    </collision>
     <inertial>
       <origin xyz="0 0 0" rpy="0 0 0"/>

Commit message: 9_4

File: src/robot_fablab/urdf/robot_fablab.xacro (robot description, xacro)
@@ -66,5 +66,5 @@
     <parent link="base_link" />
     <child link="Left_wheel" />
-    <axis xyz="0 1 0" />
+    <axis xyz="0 -1 0" />
     <dynamics damping="0.1" friction="0.1" />
   </joint>
@@ -95,5 +95,5 @@
     <parent link="base_link" />
     <child link="Right_wheel" />
-    <axis xyz="0 1 0" />
+    <axis xyz="0 -1 0" />
     <dynamics damping="0.1" friction="0.1" />
   </joint>
@@ -127,5 +127,5 @@
     <parent link="base_link" />
     <child link="Caster" />
-    <axis xyz="0 0 1" />
+    <axis xyz="0 0 -1" />
     <dynamics damping="0.1" friction="0.1" />
   </joint>

Commit message: ok

File: src/robot_fablab/urdf/robot_fablab.xacro (robot description, xacro)
@@ -14,5 +14,5 @@
     <parent link="base_footprint"/>
     <child link="base_link"/>
-    <origin xyz="0 0 0" rpy="0 0 0"/>
+    <origin xyz="0 0 0" rpy="0 0 -3.1456"/>
   </joint>
   <!-- ================= BASE LINK ================= -->
